Commit message: feat(lunar_bot): Phase D0 capability stack on the lunar base
Base, localization plumbing, MoveIt model and deploy scenes needed to run Mission A
through the real graph (research repo F50):

- Omnidirectional base: base_kinematics omni (the 4WIS crabs; SRB's term now takes
  (vx, vy, wz)); Nav2 lateral/accel/rotation limits and a 60 m global costmap derived
  from robot.yaml; `_apply_path_overrides` for dotted keys, type-preserving. Spin
  recovery at the shared 1.0 rad/s tripped the kernel's 0.5 rad/s envelope.
- LunarBot's own Nav2 and slam_toolbox base files (nav2_params_file /
  slam_params_file): voxel column below the DEM floor; 35 m laser range (latter not
  yet selected).
- New rskill-procedural-move_base_to_pose: docks on an exact planar pose with
  (vx, vy, wz), entering along the goal's axis. Live: Nav2 staging -> work pose.
- rm_75_config self-model: chassis deck/wheels/gripper/tcp_frame around the RM-75,
  chassis_base_link as planning root, the rover's 14 other joints as passive joints
  (each unknown joint logged an ERROR per /joint_states message).
- Sensor bridge: arm-mount TF; `odom_source: wheel` (4WIS least squares + IMU yaw
  rate) with the simulator pose on /openral/pose_truth for evaluation only. Default
  stays `truth` until map-based localization lands.
- lxml dependency (MoveIt launch inside the deploy graph); Mission A/B deploy scenes
  (reasoner off) plus camera-free `_fast` variants.

Co-Authored-By: Claude Opus 5 (1M context) <noreply@anthropic.com>
Claude-Session: https://claude.ai/code/session_01Rwo8Aw8ErX16wHthZQ8E9d

File: packages/rm_75_config/config/lunarbot_body.xacro (robot description, xacro)
@@ -39,4 +39,37 @@
       </collision>
     </link>
+    <!-- The rover's other actuated joints. They carry no geometry (the wheels' envelope is already on
+         chassis_base_link above and steering barely changes it), but the model must KNOW them: the robot
+         publishes one 21-joint /joint_states, and MoveIt's CurrentStateMonitor logged an ERROR per unknown
+         joint per message — ~600 lines/s, enough to drown the deploy log (research repo F50). -->
+    <xacro:macro name="passive_joint" params="name parent:=chassis_base_link axis:='0 0 1' type:=revolute lower:=-3.15 upper:=3.15">
+      <link name="${name}_link"/>
+      <joint name="${name}" type="${type}">
+        <parent link="${parent}"/>
+        <child link="${name}_link"/>
+        <origin xyz="0 0 0" rpy="0 0 0"/>
+        <axis xyz="${axis}"/>
+        <xacro:if value="${type == 'revolute'}">
+          <limit lower="${lower}" upper="${upper}" effort="0" velocity="0"/>
+        </xacro:if>
+        <xacro:if value="${type == 'continuous'}">
+          <limit effort="0" velocity="0"/>
+        </xacro:if>
+      </joint>
+    </xacro:macro>
+    <xacro:passive_joint name="chassis_to_front_left_steering_joint"/>
+    <xacro:passive_joint name="chassis_to_front_right_steering_joint"/>
+    <xacro:passive_joint name="chassis_to_rear_left_steering_joint"/>
+    <xacro:passive_joint name="chassis_to_rear_right_steering_joint"/>
+    <xacro:passive_joint name="front_left_steering_to_wheel_joint" axis="0 1 0" type="continuous"/>
+    <xacro:passive_joint name="front_right_steering_to_wheel_joint" axis="0 1 0" type="continuous"/>
+    <xacro:passive_joint name="rear_left_steering_to_wheel_joint" axis="0 1 0" type="continuous"/>
+    <xacro:passive_joint name="rear_right_steering_to_wheel_joint" axis="0 1 0" type="continuous"/>
+    <xacro:passive_joint name="eg2_joint1" parent="Link7" lower="-0.9" upper="0.9"/>
+    <xacro:passive_joint name="eg2_joint2" parent="Link7" lower="-0.9" upper="0.9"/>
+    <xacro:passive_joint name="eg2_joint3" parent="Link7" lower="-0.9" upper="0.9"/>
+    <xacro:passive_joint name="eg2_joint4" parent="Link7" lower="-0.9" upper="0.9"/>
+    <xacro:passive_joint name="eg2_joint5" parent="Link7" lower="-0.9" upper="0.9"/>
+    <xacro:passive_joint name="eg2_joint6" parent="Link7" lower="-0.9" upper="0.9"/>
     <joint name="chassis_to_arm_mount" type="fixed">
       <parent link="chassis_base_link"/>
